File: Kicad-schematic/Colorlight-5A-75E/Colorlight-5A-75E.sch (KiCad schematic (older format))
At the start: 43 parts, among them IC1 LFE5U-25F-6BG256C, J1 HUB75 port, J10 HUB75 port, J11 HUB75 port, J12 HUB75 port, J13 HUB75 port, J14 HUB75 port, J15 HUB75 port, J16 HUB75 port, J2 HUB75 port, J3 HUB75 port, J4 HUB75 port, J5 HUB75 port, J6 HUB75 port, J7 HUB75 port, J8 HUB75 port, J9 HUB75 port, U10 74HC245, U11 74HC245, U12 74HC245, U13 74HC245, U14 74HC245, U15 74HC245, U16 74HC245, U17 74HC245, U18 74HC245, U19 74HC245, U20 74HC245, U21 74HC245, U22 74HC245, U23 74HC245, U24 74HC245, U25 74HC245, U26 74HC245, U27 74HC245, U28 74HC245, U29 M12L16161A, U30 74HC245, U32 M12L16161A, U38 74HC245, U39 74HC245, U9 74HC245

Commit message: Conectores añadidos
Parts:
- added J19: Connector, symbol Connector_Generic:Conn_01x05
- added J27: JTAG: TCK, symbol Connector_Generic:Conn_01x01
- added J28: SW_Push, symbol Switch:SW_Push
- added J30: JTAG: TDO, symbol Connector_Generic:Conn_01x01
- added J31: JTAG: TMS, symbol Connector_Generic:Conn_01x01
- added J32: JTAG: TDI, symbol Connector_Generic:Conn_01x01
- added J33: 3.3V, symbol Connector_Generic:Conn_01x01
- added J34: GND, symbol Connector_Generic:Conn_01x01
- added RP1, RP10, RP11, RP12, RP13, RP14, RP15, RP16, RP17, RP18, RP19, RP2, RP20, RP21, RP22, RP23, RP24, RP25, RP26, RP27, RP28, RP29, RP3, RP30, RP31, RP32, RP33, RP34, RP35, RP36, RP37, RP38, RP39, RP4, RP40, RP41, RP42, RP43, RP44, RP45, RP46, RP5, RP6, RP7, RP8, RP9: 330, symbol Device:R_Pack03
- gave numbers to parts that had none: 1
- renumbered IC1 to U33
Connections:
- wire segments 0 -> 256

Commit message: Nomenclatura inicial para conexiones
Connections:
- net labels added: +3.3V, G3, GND, J1_1, J1_2, J1_5, J1_6, J1_7, J1_G3, J1_R_G3, Jx_B16, Jx_F12, Jx_F15, Jx_J14, Jx_J5, Jx_K1, Jx_K2, Jx_L2, PL2B, PL2C, PT11B, PT15B, PT18A, PT18B, PT22A, PT22B, PT24A, PT24B, PT27A, PT27B, PT29A, PT33A, PT35A, PT38A, PT38B, PT40A, PT40B, PT42A, PT44B, PT47A, PT47B, PT49B, PT4A, PT4B, PT51A, PT53A, PT56A, PT56B, PT60A, PT62A, SPI_CCLK, SPI_CS, SPI_MISO, SPI_MOSI, TCK, TDI, TDO, TMS, U32_A4, U32_A7, U32_A8, U32_A9, U32_B10, U32_B11, U32_B12, U32_B7, U32_B8, U32_C12, U32_C4, U32_C6, U32_C7, U32_C8, U32_D10, U32_D11, U32_D13, U32_D3, U32_D4, U32_D5, U32_D6, U32_D7, U32_D8, U32_D9, U32_E10, U32_E11, U32_E2, U32_E4, U32_E5, U32_E6, U32_E7, U32_E9
- wire segments 256 -> 547
- no-connect marks 0 -> 1
Other:
- moved on the sheet: U29, U33
